Commit message: 楼梯步态终于收敛了

File: resources/robots/m20/urdf/m20.urdf (robot description, URDF)
Before this commit: robot M20, 17 links, 16 joints
Joints:
- joint fl_hipx_joint: limit lower=-0.611 upper=0.436 effort=76.4 velocity=22.4 -> lower=-0.611 upper=0.436 effort=76.4 velocity=20
- joint fl_hipy_joint: limit lower=-2.583 upper=2.286 effort=76.4 velocity=22.4 -> lower=-2.583 upper=2.286 effort=76.4 velocity=20
- joint fl_knee_joint: limit lower=-2.792 upper=2.809 effort=76.4 velocity=22.4 -> lower=-2.792 upper=2.809 effort=76.4 velocity=20
- joint fl_wheel_joint: limit lower=-999999 upper=999999 effort=21.6 velocity=79.3 -> lower=-999999 upper=999999 effort=21.6 velocity=35
- joint fr_hipx_joint: limit lower=-0.436 upper=0.611 effort=76.4 velocity=22.4 -> lower=-0.436 upper=0.611 effort=76.4 velocity=20
- joint fr_hipy_joint: limit lower=-2.583 upper=2.286 effort=76.4 velocity=22.4 -> lower=-2.583 upper=2.286 effort=76.4 velocity=20
- joint fr_knee_joint: limit lower=-2.792 upper=2.809 effort=76.4 velocity=22.4 -> lower=-2.792 upper=2.809 effort=76.4 velocity=20
- joint fr_wheel_joint: limit lower=-999999 upper=999999 effort=21.6 velocity=79.3 -> lower=-999999 upper=999999 effort=21.6 velocity=35
- joint hl_hipx_joint: limit lower=-0.611 upper=0.436 effort=76.4 velocity=22.4 -> lower=-0.611 upper=0.436 effort=76.4 velocity=20
- joint hl_hipy_joint: limit lower=-2.286 upper=2.583 effort=76.4 velocity=22.4 -> lower=-2.286 upper=2.583 effort=76.4 velocity=20
- joint hl_knee_joint: limit lower=-2.809 upper=2.792 effort=76.4 velocity=22.4 -> lower=-2.809 upper=2.792 effort=76.4 velocity=20
- joint hl_wheel_joint: limit lower=-999999 upper=999999 effort=21.6 velocity=79.3 -> lower=-999999 upper=999999 effort=21.6 velocity=35
- joint hr_hipx_joint: limit lower=-0.436 upper=0.611 effort=76.4 velocity=22.4 -> lower=-0.436 upper=0.611 effort=76.4 velocity=20
- joint hr_hipy_joint: limit lower=-2.286 upper=2.583 effort=76.4 velocity=22.4 -> lower=-2.286 upper=2.583 effort=76.4 velocity=20
- joint hr_knee_joint: limit lower=-2.809 upper=2.792 effort=76.4 velocity=22.4 -> lower=-2.809 upper=2.792 effort=76.4 velocity=20
- joint hr_wheel_joint: limit lower=-999999 upper=999999 effort=21.6 velocity=79.3 -> lower=-999999 upper=999999 effort=21.6 velocity=35
