Commit message: b2w 可以上,姿态不对

File: resources/robots/b2w_description/urdf/b2w_description_fix.urdf (robot description, URDF)
Before this commit: robot b2w_description, 26 links, 25 joints
Joints:
- joint FL_foot_joint: limit lower=-999999 upper=999999 effort=20 velocity=50 -> lower=-999999 upper=999999 effort=20 velocity=35
- joint FR_foot_joint: limit lower=-999999 upper=999999 effort=20 velocity=50 -> lower=-999999 upper=999999 effort=20 velocity=35
- joint RL_foot_joint: limit lower=-999999 upper=999999 effort=20 velocity=50 -> lower=-999999 upper=999999 effort=20 velocity=35
- joint RR_foot_joint: limit lower=-999999 upper=999999 effort=20 velocity=50 -> lower=-999999 upper=999999 effort=20 velocity=35
